Commit message: Add wheels to robot model

File: udacity_bot/urdf/udacity_bot.xacro (robot description, xacro)
@@ -55,3 +55,65 @@
     </visual>
   </link>
+  <link name ='left_wheel'>
+    <inertial>
+      <mass value="5"/>
+      <origin xyz="0 0 0" rpy="0 1.5707 1.5707"/>
+      <inertia
+          ixx="0.1" ixy="0" ixz="0"
+          iyy="0.1" iyz="0"
+          izz="0.1"
+      />
+    </inertial>
+    <collision name='left_wheel_collision'>
+       <origin xyz="0 0 0" rpy="0 1.5707 1.5707"/>
+       <geometry>
+         <cylinder radius="0.1" length="0.05"/>
+       </geometry>
+    </collision>
+    <visual name='left_wheel_visual'>
+        <origin xyz="0 0 0" rpy="0 1.5707 1.5707"/>
+        <geometry>
+          <cylinder radius="0.1" length="0.05"/>
+        </geometry>
+    </visual>
+  </link>
+  <link name ='right_wheel'>
+    <inertial>
+      <mass value="5"/>
+      <origin xyz="0 0 0" rpy="0 1.5707 1.5707"/>
+      <inertia
+          ixx="0.1" ixy="0" ixz="0"
+          iyy="0.1" iyz="0"
+          izz="0.1"
+      />
+    </inertial>
+    <collision name='right_wheel_collision'>
+       <origin xyz="0 0 0" rpy="0 1.5707 1.5707"/>
+       <geometry>
+         <cylinder radius="0.1" length="0.05"/>
+       </geometry>
+    </collision>
+    <visual name='right_wheel_visual'>
+        <origin xyz="0 0 0" rpy="0 1.5707 1.5707"/>
+        <geometry>
+          <cylinder radius="0.1" length="0.05"/>
+        </geometry>
+    </visual>
+  </link>
+  <joint name="left_wheel_hinge" type="continuous">
+    <origin xyz="0 0.15 0" rpy="0 0 0"/>
+    <parent link="chassis"/>
+    <child link="left_wheel"/>
+    <axis xyz="0 1 0" rpy="0 0 0"/>
+    <limit effort="10000" velocity="1000"/>
+    <dynamics damping="1.0" friction="1.0"/>
+  </joint>
+  <joint name="right_wheel_hinge" type="continuous">
+    <origin xyz="0 -0.15 0" rpy="0 0 0"/>
+    <parent link="chassis"/>
+    <child link="right_wheel"/>
+    <axis xyz="0 1 0" rpy="0 0 0"/>
+    <limit effort="10000" velocity="1000"/>
+    <dynamics damping="1.0" friction="1.0"/>
+  </joint>
 </robot>

Commit message: Add front camera to robot model

File: udacity_bot/urdf/udacity_bot.xacro (robot description, xacro)
@@ -117,3 +117,31 @@
     <dynamics damping="1.0" friction="1.0"/>
   </joint>
+  <link name='camera'>
+    <inertial>
+      <mass value="0.1"/>
+      <origin xyz="0 0 0" rpy="0 0 0"/>
+      <inertia
+          ixx="1e-6" ixy="0" ixz="0"
+          iyy="1e-6" iyz="0"
+          izz="1e-6"
+      />
+    </inertial>
+    <collision>
+      <origin xyz="0 0 0" rpy="0 0 0"/>
+      <geometry>
+        <box size="0.05 0.05 0.05"/>
+      </geometry>
+    </collision>
+    <visual>
+      <origin xyz="0 0 0" rpy="0 0 0"/>
+      <geometry>
+        <box size="0.05 0.05 0.05"/>
+      </geometry>
+    </visual>
+  </link>
+  <joint name='camera_joint' type='fixed'>
+    <origin xyz="0.2 0 0" rpy="0 0 0"/>
+    <parent link="chassis"/>
+    <child link="camera"/>
+  </joint>
 </robot>

Commit message: Add hokuyo sensor to robot model

File: udacity_bot/urdf/udacity_bot.xacro (robot description, xacro)
@@ -145,3 +145,31 @@
     <child link="camera"/>
   </joint>
+  <link name="hokuyo">
+    <inertial>
+      <mass value="0.1"/>
+      <origin xyz="0 0 0" rpy="0 0 0"/>
+      <inertia
+          ixx="1e-6" ixy="0" ixz="0"
+          iyy="1e-6" iyz="0"
+          izz="1e-6"
+      />
+    </inertial>
+    <collision>
+      <origin xyz="0 0 0" rpy="0 0 0"/>
+      <geometry>
+        <box size="0.1 0.1 0.1"/>
+      </geometry>
+    </collision>
+    <visual>
+      <origin xyz="0 0 0" rpy="0 0 0"/>
+      <geometry>
+        <mesh filename="package://udacity_bot/meshes/hokuyo.dae"/>
+      </geometry>
+    </visual>
+  </link>
+  <joint name='hokuyo_joint' type='fixed'>
+    <origin xyz="0.15 0 0.1" rpy="0 0 0"/>
+    <parent link="chassis"/>
+    <child link="hokuyo"/>
+  </joint>
 </robot>
